File: PCB_Files/PCB_PlantWatering/PCB_PlantWatering.kicad_sch (KiCad schematic)
At the start: 104 parts, among them J1 Battery connection, J10 I2C Pins, J11 I2C Pins, J13 USB_C_Receptacle_USB2.0_16P, J2 LED_Strip, J3 32KHZ/SQW, J4 Solar Panel, J5 Power output, J6 Signal Socket, J9 Analog_Pin_Socket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

Commit message: added readme text
Parts:
- removed J2: LED_Strip, Connector_JST:JST_PH_B4B-PH-K_1x04_P2.00mm_Vertical, symbol Connector:Conn_01x04_Socket
- added H1, H2, H3, H4: MountingHole, MountingHole:MountingHole_3.2mm_M3, symbol Mechanical:MountingHole
- added J12: LED_Strip, Connector_JST:JST_PH_B4B-PH-K_1x04_P2.00mm_Vertical, symbol Connector:Conn_01x04_Socket
- added J2: Connector to PCB2, Connector_PinSocket_2.00mm:PinSocket_1x06_P2.00mm_Vertical, symbol Connector:Conn_01x06_Socket
- added J7: I2C, Connector_PinSocket_2.00mm:PinSocket_1x02_P2.00mm_Vertical, symbol Connector:Conn_01x02_Socket
- added J8: Power, Connector_PinSocket_2.00mm:PinSocket_1x02_P2.00mm_Vertical, symbol Connector:Conn_01x02_Socket
- added R43, R44: 4.7k, Resistor_SMD:R_1206_3216Metric, symbol Device:R_Small
- U1: now left out of the parts list
Connections:
- net +3.3V: now also J2.3 (Pin_3), J8.2 (Pin_2), R43.2, R44.2
- net +5V: now also J12.3 (Pin_3), J2.2 (Pin_2)
- net Analog10: no longer U1.6 (VDET_2/GPIO35/ADC1_CH7)
- net Analog11: no longer U1.3 (SENSOR_VP/GPIO36/ADC1_CH0)
- net Analog12: no longer U1.4 (SENSOR_VN/GPIO39/ADC1_CH3)
- net Analog9: no longer U1.5 (VDET_1/GPIO34/ADC1_CH6)
- net GND: now also J12.1 (Pin_1), J12.4 (Pin_4), J2.6 (Pin_6), J8.1 (Pin_1)
- net LCD_CS: now also U1.8 (32K_XN/GPIO33/ADC1_CH5); no longer U1.7 (32K_XP/GPIO32/ADC1_CH4)
- net LCD_D0: now also U1.13 (MTDI/GPIO12/ADC2_CH5); no longer U1.27 (GPIO16)
- net LCD_D1: now also U1.15 (MTCK/GPIO13/ADC2_CH4); no longer U1.28 (GPIO17)
- net LCD_D2: now also U1.10 (DAC_2/ADC2_CH9/GPIO26); no longer U1.9 (DAC_1/ADC2_CH8/GPIO25)
- net LCD_D3: now also U1.9 (DAC_1/ADC2_CH8/GPIO25); no longer U1.10 (DAC_2/ADC2_CH9/GPIO26)
- net LCD_D4: now also U1.28 (GPIO17); no longer U1.11 (ADC2_CH7/GPIO27)
- net LCD_D5: now also U1.27 (GPIO16); no longer U1.12 (MTMS/GPIO14/ADC2_CH6)
- net LCD_D6: now also U1.11 (ADC2_CH7/GPIO27); no longer U1.13 (MTDI/GPIO12/ADC2_CH5)
- net LCD_D7: now also U1.12 (MTMS/GPIO14/ADC2_CH6); no longer U1.15 (MTCK/GPIO13/ADC2_CH4)
- net LCD_RS: now also U1.6 (VDET_2/GPIO35/ADC1_CH7)
- net LCD_WR: now also U1.26 (ADC2_CH0/GPIO4), U1.4 (SENSOR_VN/GPIO39/ADC1_CH3); no longer U1.8 (32K_XN/GPIO33/ADC1_CH5)
- net SCL: now also J2.4 (Pin_4), J7.1 (Pin_1), R43.1
- net SDA: now also J2.5 (Pin_5), J7.2 (Pin_2), R44.1
- net VBUS_IN: now also J2.1 (Pin_1)
- new net BUTTONS: U1.3 (SENSOR_VP/GPIO36/ADC1_CH0)
- new net GAS_SENSOR: U1.5 (VDET_1/GPIO34/ADC1_CH6)
- new net LED_STRIP: J12.2 (Pin_2), U1.7 (32K_XP/GPIO32/ADC1_CH4)
