File: PCB_Files/PlantWatering_PCB02/PlantWatering_PCB02/PlantWatering_PCB02.kicad_sch (KiCad schematic)
At the start: 62 parts, among them J1 Battery connection, J10 I2C Pins, J11 I2C Pins, J2 AnalogSignals, J3 32KHZ/SQW, J4 Solar Panel, J5 Power output, J6 Signal Sockets, J7 Connector to other Board, J8 I2C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

Commit message: changed PCB01
Changed lines of the file:
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@@
 	)
 	(junction
-		(at 161.29 157.48)
-		(diameter 0)
-		(color 0 0 0 0)
-	)
-	(junction
 		(at 226.06 137.16)
 		(diameter 0)
@@
 	)
 	(junction
-		(at 161.29 165.1)
-		(diameter 0)
-		(color 0 0 0 0)
-	)
-	(junction
 		(at 241.3 34.29)
 		(diameter 0)
@@
 	(wire
 		(pts
-			(xy 161.29 157.48) (xy 163.83 157.48)
-		)
-		(stroke
-			(width 0)
-			(type default)
-		)
-	)
-	(wire
-		(pts
 			(xy 151.13 67.31) (xy 186.69 67.31)
 		)
@@
 	(wire
 		(pts
-			(xy 156.21 165.1) (xy 161.29 165.1)
+			(xy 156.21 165.1) (xy 163.83 165.1)
 		)
 		(stroke
@@
 	(wire
 		(pts
-			(xy 156.21 157.48) (xy 161.29 157.48)
+			(xy 156.21 157.48) (xy 163.83 157.48)
 		)
 		(stroke
@@
 	(wire
 		(pts
-			(xy 161.29 165.1) (xy 163.83 165.1)
-		)
-		(stroke
-			(width 0)
-			(type default)
-		)
-	)
-	(wire
-		(pts
 			(xy 172.72 125.73) (xy 181.61 125.73)
 		)
@@
 	)
 	(symbol
-		(lib_id "power:PWR_FLAG")
-		(at 161.29 165.1 0)
-		(unit 1)
-		(body_style 1)
-		(exclude_from_sim no)
-		(in_bom yes)
-		(on_board yes)
-		(in_pos_files yes)
-		(dnp no)
-		(fields_autoplaced yes)
-		(property "Reference" "#FLG02"
-			(at 161.29 163.195 0)
-			(hide yes)
-			(show_name no)
-			(do_not_autoplace no)
-			(effects
-				(font
-					(size 1.27 1.27)
-				)
-			)
-		)
-		(property "Value" "PWR_FLAG"
-			(at 161.29 160.02 0)
-			(show_name no)
-			(do_not_autoplace no)
-			(effects
-				(font
-					(size 1.27 1.27)
-				)
-			)
-		)
-		(property "Footprint" ""
-			(at 161.29 165.1 0)
-			(hide yes)
-			(show_name no)
-			(do_not_autoplace no)
-			(effects
-				(font
-					(size 1.27 1.27)
-				)
-			)
-		)
-		(property "Datasheet" ""
-			(at 161.29 165.1 0)
-			(hide yes)
-			(show_name no)
-			(do_not_autoplace no)
-			(effects
-				(font
-					(size 1.27 1.27)
-				)
-			)
-		)
-		(property "Description" "Special symbol for telling ERC where power comes from"
-			(at 161.29 165.1 0)
-			(hide yes)
-			(show_name no)
-			(do_not_autoplace no)
-			(effects
-				(font
-					(size 1.27 1.27)
-				)
-			)
-		)
-		(pin "1"
-		)
-		(instances
-			(project "PlantWatering_PCB02"
-				(path "/c5f9ebaf-06b2-436d-9d56-c191f4c0635f"
-					(reference "#FLG02")
-					(unit 1)
-				)
-			)
-		)
-	)
-	(symbol
 		(lib_name "+3.3V_3")
 		(lib_id "power:+3.3V")
@@
 					(unit 1)
 				)
-			)
-		)
-	)
-	(symbol
-		(lib_id "power:PWR_FLAG")
-		(at 161.29 157.48 0)
-		(unit 1)
-		(body_style 1)
-		(exclude_from_sim no)
-		(in_bom yes)
-		(on_board yes)
-		(in_pos_files yes)
-		(dnp no)
-		(fields_autoplaced yes)
-		(property "Reference" "#FLG01"
-			(at 161.29 155.575 0)
-			(hide yes)
-			(show_name no)
-			(do_not_autoplace no)
-			(effects
-				(font
-					(size 1.27 1.27)
-				)
-			)
-		)
-		(property "Value" "PWR_FLAG"
-			(at 161.29 152.4 0)
-			(show_name no)
-			(do_not_autoplace no)
-			(effects
-				(font
-					(size 1.27 1.27)
-				)
-			)
-		)
-		(property "Footprint" ""
-			(at 161.29 157.48 0)
-			(hide yes)
-			(show_name no)
-			(do_not_autoplace no)
-			(effects
-				(font
-					(size 1.27 1.27)
-				)
-			)
-		)
-		(property "Datasheet" ""
-			(at 161.29 157.48 0)
-			(hide yes)
-			(show_name no)
-			(do_not_autoplace no)
-			(effects
-				(font
-					(size 1.27 1.27)
-				)
-			)
-		)
-		(property "Description" "Special symbol for telling ERC where power comes from"
-			(at 161.29 157.48 0)
-			(hide yes)
-			(show_name no)
-			(do_not_autoplace no)
-			(effects
-				(font
-					(size 1.27 1.27)
-				)
-			)
-		)
-		(pin "1"
-		)
-		(instances
-			(project "PlantWatering_PCB02"
-				(path "/c5f9ebaf-06b2-436d-9d56-c191f4c0635f"
-					(reference "#FLG01")
-					(unit 1)
-				)
