File: PCB_Files/PlantWatering_PCB01/PlantWatering_PCB01/PlantWatering_PCB01.kicad_sch (KiCad schematic)
At the start: 54 parts, among them J1 Connector to PCB2, J13 USB_C_Receptacle_USB2.0_16P, J2 LED_Strip, J3 I2C, J4 Power, Q1 MUN5211DW1, SW1 SW_Push, SW2 SW_Push, SW3 SW_Push, SW4 SW_Push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

Commit message: changed PCB01
Parts:
- R1, R2: LCSC PN C23186 -> C27834
- R18, R19, R39, R9: footprint Resistor_SMD:R_1206_3216Metric -> Resistor_SMD:R_0805_2012Metric; LCSC PN C1489 -> C17414
- R3: LCSC PN C4190 -> C17520
- R7: LCSC PN C23061 -> C26011
Changed lines of the file:
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@@
 			)
 		)
-		(property "LCSC PN" "C23186"
+		(property "LCSC PN" "C27834"
 			(at 76.2 41.91 0)
 			(hide yes)
@@
 			)
 		)
-		(property "Footprint" "Resistor_SMD:R_1206_3216Metric"
+		(property "Footprint" "Resistor_SMD:R_0805_2012Metric"
 			(at 168.91 181.61 0)
 			(hide yes)
@@
 			)
 		)
-		(property "LCSC PN" "C1489"
+		(property "LCSC PN" "C17414"
 			(at 168.91 181.61 0)
 			(hide yes)
@@
 			)
 		)
-		(property "LCSC PN" "C4190"
+		(property "LCSC PN" "C17520"
 			(at 90.17 31.75 0)
 			(hide yes)
@@
 			)
 		)
-		(property "Footprint" "Resistor_SMD:R_1206_3216Metric"
+		(property "Footprint" "Resistor_SMD:R_0805_2012Metric"
 			(at 219.71 129.54 0)
 			(hide yes)
@@
 			)
 		)
-		(property "LCSC PN" "C1489"
+		(property "LCSC PN" "C17414"
 			(at 219.71 129.54 90)
 			(hide yes)
@@
 			)
 		)
-		(property "Footprint" "Resistor_SMD:R_1206_3216Metric"
+		(property "Footprint" "Resistor_SMD:R_0805_2012Metric"
 			(at 213.36 144.78 0)
 			(hide yes)
@@
 			)
 		)
-		(property "LCSC PN" "C1489"
+		(property "LCSC PN" "C17414"
 			(at 213.36 144.78 90)
 			(hide yes)
@@
 			)
 		)
-		(property "LCSC PN" "C23061"
+		(property "LCSC PN" "C26011"
 			(at 261.62 83.82 0)
 			(hide yes)
@@
 			)
 		)
-		(property "Footprint" "Resistor_SMD:R_1206_3216Metric"
+		(property "Footprint" "Resistor_SMD:R_0805_2012Metric"
 			(at 170.18 62.738 90)
 			(hide yes)
@@
 			)
 		)
-		(property "LCSC PN" "C1489"
+		(property "LCSC PN" "C17414"
 			(at 170.18 60.96 90)
 			(hide yes)
@@
 			)
 		)
-		(property "LCSC PN" "C23186"
+		(property "LCSC PN" "C27834"
 			(at 67.31 41.91 0)
 			(hide yes)

Commit message: changed resistance of buttons (look at schematic)
Parts:
- R25, R26, R27: value 1k -> 10k; footprint Resistor_SMD:R_1206_3216Metric -> Resistor_SMD:R_0805_2012Metric; LCSC PN C1469 -> C17414
- R28: value 1k -> 62k; footprint Resistor_SMD:R_1206_3216Metric -> Resistor_SMD:R_0805_2012Metric; LCSC PN C1469 -> C17783
Changed lines of the file:
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@@
 			)
 		)
-		(property "Value" "1k"
+		(property "Value" "62k"
 			(at 181.356 125.984 90)
 			(show_name no)
@@
 			)
 		)
-		(property "Footprint" "Resistor_SMD:R_1206_3216Metric"
+		(property "Footprint" "Resistor_SMD:R_0805_2012Metric"
 			(at 181.61 128.27 0)
 			(hide yes)
@@
 			)
 		)
-		(property "LCSC PN" "C1469"
+		(property "LCSC PN" "C17783"
 			(at 181.61 128.27 90)
 			(hide yes)
@@
 			)
 		)
-		(property "Value" "1k"
+		(property "Value" "10k"
 			(at 172.72 125.73 90)
 			(show_name no)
@@
 			)
 		)
-		(property "Footprint" "Resistor_SMD:R_1206_3216Metric"
+		(property "Footprint" "Resistor_SMD:R_0805_2012Metric"
 			(at 172.72 128.27 0)
 			(hide yes)
@@
 			)
 		)
-		(property "LCSC PN" "C1469"
+		(property "LCSC PN" "C17414"
 			(at 172.72 128.27 90)
 			(hide yes)
@@
 			)
 		)
-		(property "Value" "1k"
+		(property "Value" "10k"
 			(at 149.86 125.73 90)
 			(show_name no)
@@
 			)
 		)
-		(property "Footprint" "Resistor_SMD:R_1206_3216Metric"
+		(property "Footprint" "Resistor_SMD:R_0805_2012Metric"
 			(at 149.86 128.27 0)
 			(hide yes)
@@
 			)
 		)
-		(property "LCSC PN" "C1469"
+		(property "LCSC PN" "C17414"
 			(at 149.86 128.27 90)
 			(hide yes)
@@
 			)
 		)
-		(property "Value" "1k"
+		(property "Value" "10k"
 			(at 161.29 125.73 90)
 			(show_name no)
@@
 			)
 		)
-		(property "Footprint" "Resistor_SMD:R_1206_3216Metric"
+		(property "Footprint" "Resistor_SMD:R_0805_2012Metric"
 			(at 161.29 128.27 0)
 			(hide yes)
@@
 			)
 		)
-		(property "LCSC PN" "C1469"
+		(property "LCSC PN" "C17414"
 			(at 161.29 128.27 90)
 			(hide yes)
