File: PCB_Files/PlantWatering_PCB01/PlantWatering_PCB01/PlantWatering_PCB01.kicad_sch (KiCad schematic)
At the start: 54 parts, among them J1 Connector to PCB2, J13 USB_C_Receptacle_USB2.0_16P, J2 LED_Strip, J3 I2C, J4 Power, Q1 MUN5211DW1, SW1 SW_Push, SW2 SW_Push, SW3 SW_Push, SW4 SW_Push, U1 ESP32-DevKitC, U13 MQ-6, U2 CP2102N-Axx-xQFN28, U3 XC6220B331MR

Commit message: added main pwr switch to pcb01
Parts:
- added SW6: SW_SPDT, Button_Switch_THT:SW_CK_JS202011AQN_DPDT_Angled, symbol Switch:SW_SPDT
- SW1, SW2, SW3, SW4: LCSC PN (none) -> C221662
Connections:
- net VBUS renamed VBUS_con
- net VBUS_con: now also SW6.3 (C); no longer D1.2 (A), D3.4 (K)
- new net VBUS_SW: D1.2 (A), D3.4 (K), SW6.2 (B)
- no-connect marks 23 -> 24
