File: PCB_Files/PlantWatering_PCB01/PlantWatering_PCB01/PlantWatering_PCB01.kicad_pcb (KiCad board)
At the start: 2 copper layers, 109 x 55.5 mm, 54 parts, among them J1 Connector to PCB2, J13 USB_C_Receptacle_USB2.0_16P, J2 LED_Strip, J3 I2C, J4 Power, Q1 MUN5211DW1, SW1 SW_Push, SW2 SW_Push, SW3 SW_Push, SW4 SW_Push, U1 ESP32-DevKitC, U13 MQ-6, U2 CP2102N-Axx-xQFN28, U3 XC6220B331MR

Commit message: added main pwr switch to pcb01
Parts:
- added SW6: SW_SPDT, Button_Switch_THT:SW_CK_JS202011AQN_DPDT_Angled, F.Cu at (150.0, 99.1)
- moved D2 28.3 mm to (133.0, 77.7), turned to 0 degrees
- moved R3 23.3 mm to (136.6, 77.7), turned to 180 degrees
Connections:
- D1 pad 2: VBUS -> /VBUS_SW
- D3 pad 4: VBUS -> /VBUS_SW
- J13 pad A4: VBUS -> /VBUS_con
- J13 pad A9: VBUS -> /VBUS_con
- J13 pad B4: VBUS -> /VBUS_con
- J13 pad B9: VBUS -> /VBUS_con
Routing:
- net /VBUS_SW: track 0.00 -> 40.4 mm, vias 0 -> 2
- net /VBUS_con: track 0.00 -> 30.9 mm, vias 0 -> 1
- net VBUS: track 19.6 -> 0.00 mm
- net +5V: track 156.0 -> 152.4 mm
