File: src/PCB_Files/PlantWatering_PCB01/PlantWatering_PCB01/PlantWatering_PCB01.kicad_sch (KiCad schematic)
At the start: 55 parts, among them J1 Connector to PCB2, J13 USB_C_Receptacle_USB2.0_16P, J2 LED_Strip, J3 I2C, J4 Power, Q1 MUN5211DW1, SW1 SW_Push, SW2 SW_Push, SW3 SW_Push, SW4 SW_Push, SW6 SW_SPDT, U1 ESP32-DevKitC, U13 MQ-6, U2 CP2102N-Axx-xQFN28, U3 XC6220B331MR

Commit message: changed project structure
Parts:
- SW1, SW2, SW3, SW4: LCSC PN C221662 -> (none)
- SW6: LCSC PN (none) -> C221662
Changed lines of the file:
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@@
 			)
 		)
-		(property "LCSC PN" "C221662"
+		(property "LCSC PN" ""
 			(at 177.8 115.57 90)
 			(hide yes)
@@
 			)
 		)
-		(property "LCSC PN" "C221662"
+		(property "LCSC PN" ""
 			(at 166.37 115.57 90)
 			(hide yes)
@@
 			)
 		)
-		(property "LCSC PN" "C221662"
+		(property "LCSC PN" ""
 			(at 142.24 115.57 90)
 			(hide yes)
@@
 			)
 		)
+		(property "LCSC PN" "C221662"
+			(at 194.31 161.29 0)
+			(hide yes)
+			(show_name no)
+			(do_not_autoplace no)
+			(effects
+				(font
+					(size 1.27 1.27)
+				)
+			)
+		)
 		(pin "2"
 		)
@@
 			)
 		)
-		(property "LCSC PN" "C221662"
+		(property "LCSC PN" ""
 			(at 154.94 115.57 90)
 			(hide yes)
