File: src/pcb/PlantWatering_PCB01/PlantWatering_PCB01.kicad_pcb (KiCad board)
At the start: 2 copper layers, 109 x 55.5 mm, 55 parts, among them J1 Connector to PCB2, J13 USB_C_Receptacle_USB2.0_16P, J2 LED_Strip, J3 I2C, J4 Power, Q1 MUN5211DW1, SW1 SW_Push, SW2 SW_Push, SW3 SW_Push, SW4 SW_Push, SW6 SW_SPDT, U1 ESP32-DevKitC, U13 MQ-6, U2 CP2102N-Axx-xQFN28, U3 XC6220B331MR

Commit message: final state before ordering
Parts:
- R21, R24: footprint Resistor_SMD:R_1206_3216Metric -> Resistor_SMD:R_0805_2012Metric
- moved R21 2.74 mm to (69.7, 80.7), turned to 90 degrees
- moved R24 2.73 mm to (64.8, 80.8)
Routing:
- net +3.3V: track 249.8 -> 257.8 mm
Changed lines of the file:
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@@
 			)
 		)
+		(property "LCSC PN" "C221662"
+			(at 0 0 90)
+			(unlocked yes)
+			(layer "F.Fab")
+			(hide yes)
+			(effects
+				(font
+					(size 1 1)
+					(thickness 0.15)
+				)
+			)
+		)
 		(sheetname "/")
 		(sheetfile "PlantWatering_PCB01.kicad_sch")
@@
 		)
 	)
-	(footprint "Resistor_SMD:R_1206_3216Metric"
+	(footprint "Resistor_SMD:R_0805_2012Metric"
 		(layer "F.Cu")
-		(at 68.6 83.2 -90)
-		(descr "Resistor SMD 1206 (3216 Metric), square (rectangular) end terminal, IPC-7351 nominal, (Body size source: IPC-SM-782 page 72, https://www.pcb-3d.com/wordpress/wp-content/uploads/ipc-sm-782a_amendment_1_and_2.pdf)")
+		(at 69.7 80.6875 90)
+		(descr "Resistor SMD 0805 (2012 Metric), square (rectangular) end terminal, IPC-7351 nominal, (Body size source: IPC-SM-782 page 72, https://www.pcb-3d.com/wordpress/wp-content/uploads/ipc-sm-782a_amendment_1_and_2.pdf)")
 		(tags "resistor")
 		(property "Reference" "R21"
-			(at 3.8 -0.2 90)
+			(at 0 -1.65 90)
 			(layer "F.SilkS")
 			(effects
@@
 		)
 		(property "Value" "4.7k"
-			(at 0 1.83 90)
+			(at 0 1.65 90)
 			(layer "F.Fab")
 			(effects
@@
 		)
 		(property "LCSC PN" "C17673"
-			(at 0 0 270)
+			(at 0 0 90)
 			(unlocked yes)
 			(layer "F.Fab")
@@
 		(duplicate_pad_numbers_are_jumpers no)
 		(fp_line
-			(start -0.727064 0.91)
-			(end 0.727064 0.91)
+			(start -0.227064 -0.735)
+			(end 0.227064 -0.735)
 			(stroke
 				(width 0.12)
@@
 		)
 		(fp_line
-			(start -0.727064 -0.91)
-			(end 0.727064 -0.91)
+			(start -0.227064 0.735)
+			(end 0.227064 0.735)
 			(stroke
 				(width 0.12)
@@
 		)
 		(fp_rect
-			(start -2.28 -1.13)
-			(end 2.28 1.13)
+			(start -1.68 -0.95)
+			(end 1.68 0.95)
 			(stroke
 				(width 0.05)
@@
 		)
 		(fp_rect
-			(start -1.6 -0.8)
-			(end 1.6 0.8)
+			(start -1 -0.625)
+			(end 1 0.625)
 			(stroke
 				(width 0.1)
@@
 			(effects
 				(font
-					(size 0.8 0.8)
-					(thickness 0.12)
+					(size 0.5 0.5)
+					(thickness 0.08)
 				)
 			)
 		)
 		(pad "1" smd roundrect
-			(at -1.4625 0 270)
-			(size 1.125 1.75)
+			(at -0.9125 0 90)
+			(size 1.025 1.4)
 			(layers "F.Cu" "F.Mask" "F.Paste")
-			(roundrect_rratio 0.222222)
+			(roundrect_rratio 0.243902)
 			(net "/SDA")
 			(pintype "passive")
 		)
 		(pad "2" smd roundrect
-			(at 1.4625 0 270)
-			(size 1.125 1.75)
+			(at 0.9125 0 90)
+			(size 1.025 1.4)
 			(layers "F.Cu" "F.Mask" "F.Paste")
-			(roundrect_rratio 0.222222)
+			(roundrect_rratio 0.243902)
 			(net "+3.3V")
 			(pintype "passive")
 		)
 		(embedded_fonts no)
-		(model "${KICAD10_3DMODEL_DIR}/Resistor_SMD.3dshapes/R_1206_3216Metric.step"
+		(model "${KICAD10_3DMODEL_DIR}/Resistor_SMD.3dshapes/R_0805_2012Metric.step"
 			(offset
 				(xyz 0 0 0)
@@
 		(tags "Through hole socket strip THT 1x02 2.00mm single row")
 		(property "Reference" "J3"
-			(at 0 -2.5 90)
+			(at 1.829234 1.079625 180)
 			(layer "F.SilkS")
 			(effects
@@
 		)
 	)
-	(footprint "Resistor_SMD:R_1206_3216Metric"
+	(footprint "Resistor_SMD:R_0805_2012Metric"
 		(layer "F.Cu")
-		(at 66 83.2 -90)
-		(descr "Resistor SMD 1206 (3216 Metric), square (rectangular) end terminal, IPC-7351 nominal, (Body size source: IPC-SM-782 page 72, https://www.pcb-3d.com/wordpress/wp-content/uploads/ipc-sm-782a_amendment_1_and_2.pdf)")
+		(at 64.8 80.75 -90)
+		(descr "Resistor SMD 0805 (2012 Metric), square (rectangular) end terminal, IPC-7351 nominal, (Body size source: IPC-SM-782 page 72, https://www.pcb-3d.com/wordpress/wp-content/uploads/ipc-sm-782a_amendment_1_and_2.pdf)")
 		(tags "resistor")
 		(property "Reference" "R24"
-			(at 3.9 -0.2 90)
+			(at 0 -1.75 270)
 			(layer "F.SilkS")
 			(effects
@@
 		)
 		(property "Value" "4.7k"
-			(at 0 1.83 90)
+			(at 0 1.65 270)
 			(layer "F.Fab")
 			(effects
@@
 		)
 		(property "Datasheet" ""
-			(at 0 0 90)
+			(at 0 0 270)
 			(layer "F.Fab")
 			(hide yes)
@@
 		)
 		(property "Description" "Resistor, small symbol"
-			(at 0 0 90)
+			(at 0 0 270)
 			(layer "F.Fab")
 			(hide yes)
@@
 		)
 		(property "KiLib_Generator" "SMD_2terminal_chip_molded"
-			(at 0 0 90)
+			(at 0 0 270)
 			(layer "F.SilkS")
 			(hide yes)
@@
 		(duplicate_pad_numbers_are_jumpers no)
 		(fp_line
-			(start -0.727064 0.91)
-			(end 0.727064 0.91)
+			(start -0.227064 0.735)
+			(end 0.227064 0.735)
 			(stroke
 				(width 0.12)
@@
 		)
 		(fp_line
-			(start -0.727064 -0.91)
-			(end 0.727064 -0.91)
+			(start -0.227064 -0.735)
+			(end 0.227064 -0.735)
 			(stroke
 				(width 0.12)
@@
 		)
 		(fp_rect
-			(start -2.28 -1.13)
-			(end 2.28 1.13)
+			(start -1.68 -0.95)
+			(end 1.68 0.95)
 			(stroke
 				(width 0.05)
@@
 		)
 		(fp_rect
-			(start -1.6 -0.8)
-			(end 1.6 0.8)
+			(start -1 -0.625)
+			(end 1 0.625)
 			(stroke
 				(width 0.1)
@@
 		)
 		(fp_text user "${REFERENCE}"
-			(at 0 0 90)
+			(at 0 0 270)
 			(layer "F.Fab")
 			(effects
 				(font
-					(size 0.8 0.8)
-					(thickness 0.12)
+					(size 0.5 0.5)
+					(thickness 0.08)
 				)
 			)
 		)
 		(pad "1" smd roundrect
-			(at -1.4625 0 270)
-			(size 1.125 1.75)
+			(at -0.9125 0 270)
+			(size 1.025 1.4)
 			(layers "F.Cu" "F.Mask" "F.Paste")
-			(roundrect_rratio 0.222222)
+			(roundrect_rratio 0.243902)
 			(net "/SCL")
 			(pintype "passive")
 		)
 		(pad "2" smd roundrect
-			(at 1.4625 0 270)
-			(size 1.125 1.75)
+			(at 0.9125 0 270)
+			(size 1.025 1.4)
 			(layers "F.Cu" "F.Mask" "F.Paste")
-			(roundrect_rratio 0.222222)
+			(roundrect_rratio 0.243902)
 			(net "+3.3V")
 			(pintype "passive")
 		)
 		(embedded_fonts no)
-		(model "${KICAD10_3DMODEL_DIR}/Resistor_SMD.3dshapes/R_1206_3216Metric.step"
+		(model "${KICAD10_3DMODEL_DIR}/Resistor_SMD.3dshapes/R_0805_2012Metric.step"
 			(offset
 				(xyz 0 0 0)
@@
 			)
 		)
-		(property "LCSC PN" "C221662"
+		(property "LCSC PN" ""
 			(at 0 0 180)
 			(unlocked yes)
@@
 			)
 		)
-		(property "LCSC PN" "C221662"
+		(property "LCSC PN" ""
 			(at 0 0 180)
 			(unlocked yes)
@@
 			)
 		)
-		(property "LCSC PN" "C221662"
+		(property "LCSC PN" ""
 			(at 0 0 180)
 			(unlocked yes)
@@
 			)
 		)
-		(property "LCSC PN" "C221662"
+		(property "LCSC PN" ""
 			(at 0 0 180)
 			(unlocked yes)
@@
 	)
 	(gr_text "SCL"
-		(at 65.020375 81 90)
+		(at 63.1 78.5 90)
 		(layer "F.SilkS")
 		(effects
@@
 	)
 	(gr_text "SDA"
-		(at 67 81 90)
+		(at 69.2 78.45 90)
 		(layer "F.SilkS")
 		(effects
@@
 	)
 	(segment
-		(start 66 84.6625)
-		(end 68.6 84.6625)
+		(start 64.2375 81.1)
+		(end 64.8 81.6625)
 		(width 0.5)
 		(layer "F.Cu")
@@
 	)
 	(segment
+		(start 142.925 111.575)
+		(end 144 110.5)
+		(width 0.3)
+		(layer "F.Cu")
+		(net "+3.3V")
+	)
+	(segment
 		(start 54.05 82.39939)
-		(end 54.05 92.579844)
+		(end 55.34939 81.1)
 		(width 0.5)
 		(layer "F.Cu")
@@
 	)
 	(segment
-		(start 142.925 111.575)
-		(end 144 110.5)
-		(width 0.3)
+		(start 64.8 81.6625)
+		(end 66.9875 83.85)
+		(width 0.5)
 		(layer "F.Cu")
 		(net "+3.3V")
@@
 	)
 	(segment
-		(start 66.520375 127.479234)
-		(end 66.520375 126.299234)
+		(start 71.85 81.225)
+		(end 70.4 79.775)
 		(width 0.5)
 		(layer "F.Cu")
@@
 	)
 	(segment
-		(start 62.4375 81.1)
-		(end 55.34939 81.1)
+		(start 66.520375 127.479234)
+		(end 66.520375 126.299234)
 		(width 0.5)
 		(layer "F.Cu")
@@
 	)
 	(segment
-		(start 54.05 92.579844)
-		(end 54.89939 93.429234)
+		(start 71.85 83.410661)
+		(end 71.85 81.225)
 		(width 0.5)
 		(layer "F.Cu")
@@
 	)
 	(segment
-		(start 55.34939 81.1)
-		(end 54.05 82.39939)
+		(start 71.410661 83.85)
+		(end 71.85 83.410661)
 		(width 0.5)
 		(layer "F.Cu")
@@
 	)
 	(segment
-		(start 66 84.6625)
-		(end 62.4375 81.1)
+		(start 65.545375 93.429234)
+		(end 54.89939 93.429234)
 		(width 0.5)
 		(layer "F.Cu")
@@
 	)
 	(segment
-		(start 65.545375 93.429234)
-		(end 54.89939 93.429234)
+		(start 54.89939 93.429234)
+		(end 54.05 92.579844)
+		(width 0.5)
+		(layer "F.Cu")
+		(net "+3.3V")
+	)
+	(segment
+		(start 66.9875 83.85)
+		(end 71.410661 83.85)
 		(width 0.5)
 		(layer "F.Cu")
@@
 	)
 	(segment
+		(start 55.34939 81.1)
+		(end 64.2375 81.1)
+		(width 0.5)
+		(layer "F.Cu")
+		(net "+3.3V")
+	)
+	(segment
 		(start 114.245766 127.179234)
 		(end 119.825 121.6)
@@
 	)
 	(segment
+		(start 70.4 79.775)
+		(end 69.7 79.775)
+		(width 0.5)
+		(layer "F.Cu")
+		(net "+3.3V")
+	)
+	(segment
 		(start 140.2 104.9)
 		(end 140.2 105.65)
@@
 	)
 	(segment
+		(start 54.05 92.579844)
+		(end 54.05 82.39939)
+		(width 0.5)
+		(layer "F.Cu")
+		(net "+3.3V")
+	)
+	(segment
 		(start 139.8 106.05)
 		(end 142.275 106.05)
@@
 	)
 	(segment
-		(start 53.2 82.259441)
-		(end 57.980207 77.479234)
+		(start 71.1 83.1)
+		(end 68.0625 83.1)
 		(width 0.5)
 		(layer "F.Cu")
@@
 	)
 	(segment
-		(start 67.3625 83.1)
-		(end 66 81.7375)
+		(start 64.8 79.8375)
+		(end 64.8 77.758859)
 		(width 0.5)
 		(layer "F.Cu")
@@
 	)
 	(segment
-		(start 64.520375 77.479234)
-		(end 64.520375 80.257875)
+		(start 53.2 82.259441)
+		(end 57.980207 77.479234)
 		(width 0.5)
 		(layer "F.Cu")
@@
 	)
 	(segment
-		(start 64.520375 80.257875)
-		(end 66 81.7375)
+		(start 127.704039 128.6)
+		(end 129.2 128.6)
 		(width 0.5)
 		(layer "F.Cu")
@@
 	)
 	(segment
-		(start 127.704039 128.6)
-		(end 129.2 128.6)
+		(start 68.0625 83.1)
+		(end 64.8 79.8375)
 		(width 0.5)
 		(layer "F.Cu")
@@
 	)
 	(segment
-		(start 71.1 83.1)
-		(end 67.3625 83.1)
+		(start 64.8 77.758859)
+		(end 64.520375 77.479234)
 		(width 0.5)
 		(layer "F.Cu")
