File: src/pcb/PlantWatering_PCB01/PlantWatering_PCB01.kicad_sch (KiCad schematic)
At the start: 55 parts, among them J1 Connector to PCB2, J13 USB_C_Receptacle_USB2.0_16P, J2 LED_Strip, J3 I2C, J4 Power, Q1 MUN5211DW1, SW1 SW_Push, SW2 SW_Push, SW3 SW_Push, SW4 SW_Push, SW6 SW_SPDT, U1 ESP32-DevKitC, U13 MQ-6, U2 CP2102N-Axx-xQFN28, U3 XC6220B331MR

Commit message: changed structure
Other:
- company: (none) -> benedikt314159
- title: (none) -> SmartIrrigationSystem
Changed lines of the file:
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@@
 	(generator_version "10.0")
 	(paper "A4")
+	(title_block
+		(title "SmartIrrigationSystem")
+		(date "2026-07-05")
+		(rev "V1.1")
+		(company "benedikt314159")
+	)
 	(text "Candidates:\nMUN5211DW1\nUMH3NTN\n"
 		(exclude_from_sim no)

Commit message: final state before ordering
Parts:
- R21, R24: footprint Resistor_SMD:R_1206_3216Metric -> Resistor_SMD:R_0805_2012Metric
Changed lines of the file:
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@@
 			)
 		)
-		(property "Footprint" "Resistor_SMD:R_1206_3216Metric"
+		(property "Footprint" "Resistor_SMD:R_0805_2012Metric"
 			(at 109.22 162.56 0)
 			(hide yes)
@@
 			)
 		)
-		(property "Footprint" "Resistor_SMD:R_1206_3216Metric"
+		(property "Footprint" "Resistor_SMD:R_0805_2012Metric"
 			(at 109.22 158.75 0)
 			(hide yes)

Commit message: I ordered it!!!!!
Parts:
- U2: LCSC PN C969151 -> C964632
Changed lines of the file:
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@@
 			)
 		)
-		(property "LCSC PN" "C969151"
+		(property "LCSC PN" "C964632"
 			(at 138.43 52.07 0)
 			(hide yes)
