File: src/pcb/PlantWatering_PCB02/PlantWatering_PCB02.kicad_pcb (KiCad board)
At the start: 2 copper layers, 109 x 55.5 mm, 62 parts, among them J1 Battery connection, J10 I2C Pins, J11 I2C Pins, J2 AnalogSignals, J3 32KHZ/SQW, J4 Solar Panel, J5 Power output, J6 Signal Sockets, J7 Connector to other Board, J8 I2C, J9 PWR_Output, U10 DS3231MZ, U11 TP4056-42-ESOP8, U12 AT24CS32-SSHM, U14 MT3608, U4 BMP280, U5 ADS1115IDGS, U6 ADS1115IDGS, U7 CCS811, U8 DW01A, U9 FS8205A

Commit message: final state before ordering
Parts:
- removed C8: 0.1uF, Capacitor_SMD:C_0805_2012Metric
- removed C9: 1uF, Capacitor_SMD:C_0603_1608Metric
- removed R12, R13, R14, R15: 10k, Resistor_SMD:R_1206_3216Metric
- removed U4: BMP280, Package_LGA:Bosch_LGA-8_2x2.5mm_P0.65mm_ClockwisePinNumbering
- added J12: Conn_01x06_Socket, Connector_PinHeader_2.00mm:PinHeader_1x06_P2.00mm_Vertical, F.Cu at (72.7, 107.7)
Routing:
- net +3.3V: track 369.5 -> 343.8 mm
- net /SCL: track 205.5 -> 228.6 mm
- net GND: track 88.3 -> 76.4 mm, vias 22 -> 20
- net Net-(U4-CSB): track 4.86 -> 0.00 mm
- net Net-(U4-SDO): track 2.53 -> 0.00 mm
- net /SDA: track 234.1 -> 235.7 mm
