File: src/pcb/PlantWatering_PCB02/PlantWatering_PCB02.kicad_sch (KiCad schematic)
At the start: 62 parts, among them J1 Battery connection, J10 I2C Pins, J11 I2C Pins, J2 AnalogSignals, J3 32KHZ/SQW, J4 Solar Panel, J5 Power output, J6 Signal Sockets, J7 Connector to other Board, J8 I2C, J9 PWR_Output, U10 DS3231MZ, U11 TP4056-42-ESOP8, U12 AT24CS32-SSHM, U14 MT3608, U4 BMP280, U5 ADS1115IDGS, U6 ADS1115IDGS, U7 CCS811, U8 DW01A, U9 FS8205A

Commit message: changed structure and added cart
Parts:
- AudioJack1, AudioJack2, AudioJack3, AudioJack4, AudioJack5, AudioJack6, U7: now left out of the parts list
Changed lines of the file:
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@@
 	(title_block
 		(title "PlantWatering PCB02")
-		(date "2026-05-26")
-		(rev "V0")
+		(date "2026-07-05")
+		(rev "V1.1")
 		(company "@benedikt314159")
 	)
@@
 		(body_style 1)
 		(exclude_from_sim no)
-		(in_bom yes)
+		(in_bom no)
 		(on_board yes)
 		(in_pos_files yes)
@@
 		(body_style 1)
 		(exclude_from_sim no)
-		(in_bom yes)
+		(in_bom no)
 		(on_board yes)
 		(in_pos_files yes)
@@
 		(body_style 1)
 		(exclude_from_sim no)
-		(in_bom yes)
+		(in_bom no)
 		(on_board yes)
 		(in_pos_files yes)
@@
 		(body_style 1)
 		(exclude_from_sim no)
-		(in_bom yes)
+		(in_bom no)
 		(on_board yes)
 		(in_pos_files yes)
@@
 		(body_style 1)
 		(exclude_from_sim no)
-		(in_bom yes)
+		(in_bom no)
 		(on_board yes)
 		(in_pos_files yes)
@@
 		(body_style 1)
 		(exclude_from_sim no)
-		(in_bom yes)
+		(in_bom no)
 		(on_board yes)
 		(in_pos_files yes)
@@
 		(body_style 1)
 		(exclude_from_sim no)
-		(in_bom yes)
+		(in_bom no)
 		(on_board yes)
 		(in_pos_files yes)

Commit message: some improvements in order to make it cheaper (affordable)
Parts:
- AudioJack1, AudioJack2, AudioJack3, AudioJack4, AudioJack5, AudioJack6: now in the parts list
Changed lines of the file:
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@@
 		(body_style 1)
 		(exclude_from_sim no)
-		(in_bom no)
+		(in_bom yes)
 		(on_board yes)
 		(in_pos_files yes)
@@
 		(body_style 1)
 		(exclude_from_sim no)
-		(in_bom no)
+		(in_bom yes)
 		(on_board yes)
 		(in_pos_files yes)
@@
 		(body_style 1)
 		(exclude_from_sim no)
-		(in_bom no)
+		(in_bom yes)
 		(on_board yes)
 		(in_pos_files yes)
@@
 		(body_style 1)
 		(exclude_from_sim no)
-		(in_bom no)
+		(in_bom yes)
 		(on_board yes)
 		(in_pos_files yes)
@@
 		(body_style 1)
 		(exclude_from_sim no)
-		(in_bom no)
+		(in_bom yes)
 		(on_board yes)
 		(in_pos_files yes)
@@
 		(body_style 1)
 		(exclude_from_sim no)
-		(in_bom no)
+		(in_bom yes)
 		(on_board yes)
 		(in_pos_files yes)

Commit message: final state before ordering
Parts:
- removed C8: 0.1uF, Capacitor_SMD:C_0805_2012Metric, symbol Device:C_Small
- removed C9: 1uF, Capacitor_SMD:C_0603_1608Metric, symbol Device:C_Small
- removed R12, R13, R14, R15: 10k, Resistor_SMD:R_1206_3216Metric, symbol Device:R_Small
- removed U4: BMP280, Package_LGA:Bosch_LGA-8_2x2.5mm_P0.65mm_ClockwisePinNumbering, symbol Sensor_Pressure:BMP280
- added J12: Conn_01x06_Socket, Connector_PinHeader_2.00mm:PinHeader_1x06_P2.00mm_Vertical, symbol Connector:Conn_01x06_Socket
Connections:
- net +3.3V: now also J12.1 (Pin_1)
- net GND: now also J12.2 (Pin_2)
- net SCL: now also J12.3 (Pin_3)
- net SDA: now also J12.4 (Pin_4)
- no-connect marks 20 -> 22
