File: src/pcb/Smart_Irrigation_SystemV2/Smart_Irrigation_SystemV2.kicad_sch (KiCad schematic)
At the start: 134 parts, among them CN1 PJ-3136-3A, CN2 PJ-3136-3A, CN3 PJ-3136-3A, CN4 PJ-3136-3A, CN5 PJ-3136-3A, CN6 PJ-3136-3A, J1 USB_C_Receptacle_USB2.0_16P, J10 I2C, J11 I2C, J13 I2C, J14 SolarPanel, J15 I2C, J16 GPIO_Expander, J2 FPC_Connector, J6 I2C, J9 Battary Connection, Q1 MUN5211DW1, Q2 FDN340P, Q3 AO3400A, SW1 IO0 Switch, SW2 EN Switch, SW3 SW_Push, SW4 SW_Push, SW5 SW_Push, SW6 SW_Push, U1 CP2102N-Axx-xQFN28, U10 ADS1115IDGS, U11 PCA9536DP, U2 ESP32-WROOM-32, U3 ADS1115IDGS, U4 DS3231MZ, U5 TLV62568ADRL, U6 SN74LVC245APW, U7 TP4056-42-ESOP8, U8 TPS63001

Commit message: fpc connector was in the wrong orientation. I moved it to the front, made a hole into the pcb, reorganized the libraries, rerouted everything, removed the unnecessary I2C outputs, rearranged components. Still need to work on the silkscreen, 3D models, move all other components to the front. time spend: 3h
Parts:
- removed CN1, CN2, CN3, CN4, CN5, CN6: PJ-3136-3A, C707248:AUDIO-TH_PJ-3136-3A, symbol easyeda2kicad:PJ-3136-3A
- removed J2: FPC_Connector, 5051105091:CON_5051105091_MOL, symbol Connector:Conn_01x50_Socket
- added CN1, CN2, CN3, CN4, CN5, CN6: PJ-3136-3A, C707248:AUDIO-TH_PJ-3136-3A, symbol C707248:PJ-3136-3A
- added FPC2: FPC-05FB-50PH20, C2856838:FPC-SMD_50P-P0.50_FPC-05FB-50PH20, symbol easyeda2kicad:FPC-05FB-50PH20
Connections:
- net +3.3V: now also CN1.2, CN2.2, CN3.2, CN4.2, CN5.2, CN6.2, FPC2.40, FPC2.41, FPC2.42
- net GND: now also CN1.1, CN2.1, CN3.1, CN4.1, CN5.1, CN6.1, FPC2.11, FPC2.12, FPC2.13, FPC2.14, FPC2.15, FPC2.16, FPC2.17, FPC2.18, FPC2.19, FPC2.20, FPC2.21, FPC2.22, FPC2.23, FPC2.24, FPC2.34, FPC2.43, FPC2.50, FPC2.51, FPC2.52, FPC2.6, FPC2.7, FPC2.8, FPC2.9
- net GPIO14: now also FPC2.25, FPC2.45
- net GPIO15: now also FPC2.37, FPC2.44
- net GPIO27: now also FPC2.26, FPC2.46
- net GPIO33: now also FPC2.38
- net GPIO39: now also FPC2.36, FPC2.47
- net MS1: now also CN1.4
- net MS2: now also CN2.4
- net MS3: now also CN3.4
- net MS4: now also CN4.4
- net MS5: now also CN5.4
- net MS6: now also CN6.4
- net at Q3.2 (S), R38.2, TP10.1: now also FPC2.1
- net at R12.2: now also FPC2.4
- net at R15.2: now also FPC2.49
- net at R14.2: now also FPC2.48
- net at R17.2: now also FPC2.35
- net at R10.2: now also FPC2.2
- net at R11.2: now also FPC2.3
- net at R16.2: now also FPC2.10
- net at U6.13 (B6): now also FPC2.27
- net at U6.14 (B5): now also FPC2.28
- net at U6.15 (B4): now also FPC2.29
- net at U6.16 (B3): now also FPC2.30
- net at U6.17 (B2): now also FPC2.31
- net at U6.18 (B1): now also FPC2.32
- net at R13.2: now also FPC2.5

Commit message: added 3d Models
Parts:
- removed J10, J11, J13, J6: I2C, Connector_JST:JST_EH_B4B-EH-A_1x04_P2.50mm_Vertical, symbol Connector:Conn_01x04_Socket
- removed TP14: GND, TestPoint:TestPoint_Pad_D1.5mm, symbol Connector:TestPoint
- TP16: footprint TestPoint:TestPoint_Pad_4.0x4.0mm -> TestPoint:TestPoint_Pad_2.5x2.5mm

Commit message: moved silkscreen and replaced buttons with smd ones
Parts:
- SW3, SW4, SW5, SW6: footprint C83206:KEY-SMD_4P-L6.0-W6.0-P3.90-LS9.0 -> Button_Switch_THT:SW_PUSH_6mm_H5mm
Changed lines of the file:
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@@
 			)
 		)
-		(property "Footprint" "C83206:KEY-SMD_4P-L6.0-W6.0-P3.90-LS9.0"
+		(property "Footprint" "Button_Switch_THT:SW_PUSH_6mm_H5mm"
 			(at 240.03 133.35 0)
 			(hide yes)
@@
 			)
 		)
-		(property "Footprint" "C83206:KEY-SMD_4P-L6.0-W6.0-P3.90-LS9.0"
+		(property "Footprint" "Button_Switch_THT:SW_PUSH_6mm_H5mm"
 			(at 240.03 151.13 0)
 			(hide yes)
@@
 			)
 		)
-		(property "Footprint" "C83206:KEY-SMD_4P-L6.0-W6.0-P3.90-LS9.0"
+		(property "Footprint" "Button_Switch_THT:SW_PUSH_6mm_H5mm"
 			(at 240.03 124.46 0)
 			(hide yes)
@@
 			)
 		)
-		(property "Footprint" "C83206:KEY-SMD_4P-L6.0-W6.0-P3.90-LS9.0"
+		(property "Footprint" "Button_Switch_THT:SW_PUSH_6mm_H5mm"
 			(at 240.03 142.24 0)
 			(hide yes)
